Commit message: Use MikataArm model

File: open_manipulator_description/urdf/open_manipulator.urdf.xacro (robot description, xacro)
@@ -31,14 +31,14 @@
   <link name="link1">
     <visual>
-      <origin xyz="0 0 0" rpy="0 0 0"/>
-      <geometry>
-        <mesh filename="package://open_manipulator_description/meshes/chain_link1.stl" scale="0.001 0.001 0.001"/>
-      </geometry>
-      <material name="grey"/>
-    </visual>
-    <collision>
-      <origin xyz="0 0 0" rpy="0 0 0"/>
-      <geometry>
-        <mesh filename="package://open_manipulator_description/meshes/chain_link1.stl" scale="0.001 0.001 0.001"/>
+      <origin xyz="0 0 0" rpy="0 0 ${-pi*0.5}"/>
+      <geometry>
+        <mesh filename="package://open_manipulator_description/meshes/chain_link1.stl"/>
+      </geometry>
+      <material name="grey"/>
+    </visual>
+    <collision>
+      <origin xyz="0 0 0" rpy="0 0 ${-pi*0.5}"/>
+      <geometry>
+        <mesh filename="package://open_manipulator_description/meshes/chain_link1.stl"/>
       </geometry>
     </collision>
@@ -62,7 +62,7 @@
     <parent link="link1"/>
     <child link="link2"/>
-    <origin xyz="0.012 0.0 0.017" rpy="0 0 0"/>
+    <origin xyz="0 0 0.0355" rpy="0 0 0"/>
     <axis xyz="0 0 1"/>
-    <limit velocity="4.8" effort="1" lower="${-pi*0.9}" upper="${pi*0.9}" />
+    <limit velocity="4.8" effort="1" lower="${-pi}" upper="${pi}" />
   </joint>
   <!-- Transmission 1 -->
@@ -71,14 +71,14 @@
   <link name="link2">
     <visual>
-      <origin xyz="0 0 0.019" rpy="0 0 0"/>
-      <geometry>
-        <mesh filename="package://open_manipulator_description/meshes/chain_link2.stl" scale="0.001 0.001 0.001"/>
-      </geometry>
-      <material name="grey"/>
-    </visual>
-    <collision>
-      <origin xyz="0 0 0.019" rpy="0 0 0"/>
-      <geometry>
-        <mesh filename="package://open_manipulator_description/meshes/chain_link2.stl" scale="0.001 0.001 0.001"/>
+      <origin xyz="0 0 0.0405" rpy="${pi*0.5} 0 ${pi*0.5}"/>
+      <geometry>
+        <mesh filename="package://open_manipulator_description/meshes/chain_link2.stl"/>
+      </geometry>
+      <material name="grey"/>
+    </visual>
+    <collision>
+      <origin xyz="0 0 0.0405" rpy="${pi*0.5} 0 ${pi*0.5}"/>
+      <geometry>
+        <mesh filename="package://open_manipulator_description/meshes/chain_link2.stl"/>
       </geometry>
     </collision>
@@ -102,7 +102,7 @@
     <parent link="link2"/>
     <child link="link3"/>
-    <origin xyz="0.0 0.0 0.0595" rpy="0 0 0"/>
+    <origin xyz="0 0 0.0405" rpy="0 0 0"/>
     <axis xyz="0 1 0"/>
-    <limit velocity="4.8" effort="1" lower="${-pi*0.57}" upper="${pi*0.5}" />
+    <limit velocity="4.8" effort="1" lower="-1.85" upper="2.07" />
   </joint>
   <!-- Transmission 2 -->
@@ -111,14 +111,14 @@
   <link name="link3">
     <visual>
-      <origin xyz="0 0 0" rpy="0 0 0"/>
-      <geometry>
-        <mesh filename="package://open_manipulator_description/meshes/chain_link3.stl" scale="0.001 0.001 0.001"/>
-      </geometry>
-      <material name="grey"/>
-    </visual>
-    <collision>
-      <origin xyz="0 0 0" rpy="0 0 0"/>
-      <geometry>
-        <mesh filename="package://open_manipulator_description/meshes/chain_link3.stl" scale="0.001 0.001 0.001"/>
+      <origin xyz="0.024 0 0.148" rpy="0 0 ${-pi*0.5}"/>
+      <geometry>
+        <mesh filename="package://open_manipulator_description/meshes/chain_link3.stl"/>
+      </geometry>
+      <material name="grey"/>
+    </visual>
+    <collision>
+      <origin xyz="0.024 0 0.148" rpy="0 0 ${-pi*0.5}"/>
+      <geometry>
+        <mesh filename="package://open_manipulator_description/meshes/chain_link3.stl"/>
       </geometry>
     </collision>
@@ -142,7 +142,7 @@
     <parent link="link3"/>
     <child link="link4"/>
-    <origin xyz="0.024 0 0.128" rpy="0 0 0"/>
+    <origin xyz="0.024 0 0.148" rpy=" 0 0 0"/>
     <axis xyz="0 1 0"/>
-    <limit velocity="4.8" effort="1" lower="${-pi*0.3}" upper="${pi*0.44}" />
+    <limit velocity="4.8" effort="1" lower="-1.85" upper="1.41" />
   </joint>
   <!-- Transmission 3 -->
@@ -151,14 +151,14 @@
   <link name="link4">
     <visual>
-      <origin xyz="0 0 0" rpy="0 0 0"/>
-      <geometry>
-        <mesh filename="package://open_manipulator_description/meshes/chain_link4.stl" scale="0.001 0.001 0.001"/>
-      </geometry>
-      <material name="grey"/>
-    </visual>
-    <collision>
-      <origin xyz="0 0 0" rpy="0 0 0"/>
-      <geometry>
-        <mesh filename="package://open_manipulator_description/meshes/chain_link4.stl" scale="0.001 0.001 0.001"/>
+      <origin xyz="0.150 0 0" rpy="0 ${pi} ${-pi*0.5}"/>
+      <geometry>
+        <mesh filename="package://open_manipulator_description/meshes/chain_link4.stl"/>
+      </geometry>
+      <material name="grey"/>
+    </visual>
+    <collision>
+      <origin xyz="0.150 0 0" rpy="0 ${pi} ${-pi*0.5}"/>
+      <geometry>
+        <mesh filename="package://open_manipulator_description/meshes/chain_link4.stl"/>
       </geometry>
     </collision>
@@ -182,7 +182,7 @@
     <parent link="link4"/>
     <child link="link5"/>
-    <origin xyz="0.124 0.0 0.0" rpy="0 0 0"/>
+    <origin xyz="0.150 0 0" rpy="0 0 0"/>
     <axis xyz="0 1 0"/>
-    <limit velocity="4.8" effort="1" lower="${-pi*0.57}" upper="${pi*0.65}" />
+    <limit velocity="4.8" effort="1" lower="-1.64" upper="1.78" />
   </joint>
   <!-- Transmission 4 -->
@@ -193,12 +193,12 @@
       <origin xyz="0 0 0" rpy="0 0 0"/>
       <geometry>
-        <mesh filename="package://open_manipulator_description/meshes/chain_link5.stl" scale="0.001 0.001 0.001"/>
-      </geometry>
-      <material name="grey"/>
-    </visual>
-    <collision>
-      <origin xyz="0 0 0" rpy="0 0 0"/>
-      <geometry>
-        <mesh filename="package://open_manipulator_description/meshes/chain_link5.stl" scale="0.001 0.001 0.001"/>
+        <mesh filename="package://open_manipulator_description/meshes/chain_link5.stl"/>
+      </geometry>
+      <material name="grey"/>
+    </visual>
+    <collision>
+      <origin xyz="0 0 0" rpy="0 0 0"/>
+      <geometry>
+        <mesh filename="package://open_manipulator_description/meshes/chain_link5.stl"/>
       </geometry>
     </collision>
@@ -221,14 +221,14 @@
   <link name="gripper_link">
     <visual>
-      <origin xyz="0.0 0.0 0" rpy="0 0 0"/>
-      <geometry>
-        <mesh filename="package://open_manipulator_description/meshes/chain_link_grip_l.stl" scale="0.001 0.001 0.001"/>
-      </geometry>
-      <material name="grey"/>
-    </visual>
-    <collision>
-      <origin xyz="0.0 0.0 0" rpy="0 0 0"/>
-      <geometry>
-        <mesh filename="package://open_manipulator_description/meshes/chain_link_grip_l.stl" scale="0.001 0.001 0.001"/>
+      <origin xyz="0 0 0" rpy="0 0 0"/>
+      <geometry>
+        <mesh filename="package://open_manipulator_description/meshes/chain_link_grip_l.stl"/>
+      </geometry>
+      <material name="grey"/>
+    </visual>
+    <collision>
+      <origin xyz="0 0 0" rpy="0 0 0"/>
+      <geometry>
+        <mesh filename="package://open_manipulator_description/meshes/chain_link_grip_l.stl"/>
       </geometry>
     </collision>
@@ -248,11 +248,11 @@
     </inertial>-->
   </link>
-  <!--  Gripper joint -->
-  <joint name="gripper" type="prismatic">
+  <!--  Grip joint -->
+  <joint name="grip_joint" type="revolute">
     <parent link="link5"/>
-    <child link="gripper_link"/>
-    <origin xyz="0.0817 0.021 0.0" rpy="0 0 0"/>
-    <axis xyz="0 1 0"/>
-    <limit velocity="4.8" effort="1" lower="-0.010" upper="0.019" />
+    <child link="grip_link"/>
+    <origin xyz="0.04225 0.015 0" rpy="0 0 0"/>
+    <axis xyz="0 0 1"/>
+    <limit velocity="4.8" effort="1" lower="-0.7133010663668231" upper="1.059980724428978" />
   </joint>
   <!-- Transmission 5 -->
@@ -261,14 +261,14 @@
   <link name="gripper_link_sub">
     <visual>
-      <origin xyz="0.0 -0.0 0" rpy="0 0 0"/>
-      <geometry>
-        <mesh filename="package://open_manipulator_description/meshes/chain_link_grip_r.stl" scale="0.001 0.001 0.001"/>
-      </geometry>
-      <material name="grey"/>
-    </visual>
-    <collision>
-      <origin xyz="0.0 -0.0 0" rpy="0 0 0"/>
-      <geometry>
-        <mesh filename="package://open_manipulator_description/meshes/chain_link_grip_r.stl" scale="0.001 0.001 0.001"/>
+      <origin xyz="0 0 0" rpy="0 0 0"/>
+      <geometry>
+        <mesh filename="package://open_manipulator_description/meshes/chain_link_grip_r.stl"/>
+      </geometry>
+      <material name="grey"/>
+    </visual>
+    <collision>
+      <origin xyz="0 0 0" rpy="0 0 0"/>
+      <geometry>
+        <mesh filename="package://open_manipulator_description/meshes/chain_link_grip_r.stl"/>
       </geometry>
     </collision>
@@ -288,12 +288,12 @@
     </inertial>-->
   </link>
-  <!--  Gripper joint sub -->
-  <joint name="gripper_sub" type="prismatic">
+  <!--  Grip joint sub -->
+  <joint name="grip_joint_sub" type="revolute">
     <parent link="link5"/>
-    <child link="gripper_link_sub"/>
-    <origin xyz="0.0817 -0.021 0" rpy="0 0 0"/>
-    <axis xyz="0 -1 0"/>
-    <limit velocity="4.8" effort="1" lower="-0.010" upper="0.019" />
-    <mimic joint="gripper" multiplier="1"/>
+    <child link="grip_link_sub"/>
+    <origin xyz="0.04225 -0.015 0" rpy="0 0 0"/>
+    <axis xyz="0 0 1"/>
+    <limit velocity="4.8" effort="1" lower="-0.7133010663668231" upper="1.059980724428978" />
+    <mimic joint="grip_joint" multiplier="-1"/>
   </joint>
   <!-- Transmission 6 -->

Commit message: Fix link name in urdf

File: open_manipulator_description/urdf/open_manipulator.urdf.xacro (robot description, xacro)
@@ -248,8 +248,8 @@
     </inertial>-->
   </link>
-  <!--  Grip joint -->
-  <joint name="grip_joint" type="revolute">
+  <!--  Gripper joint -->
+  <joint name="gripper" type="revolute">
     <parent link="link5"/>
-    <child link="grip_link"/>
+    <child link="gripper_link"/>
     <origin xyz="0.04225 0.015 0" rpy="0 0 0"/>
     <axis xyz="0 0 1"/>
@@ -288,12 +288,12 @@
     </inertial>-->
   </link>
-  <!--  Grip joint sub -->
-  <joint name="grip_joint_sub" type="revolute">
+  <!--  Gripper joint sub -->
+  <joint name="gripper_sub" type="revolute">
     <parent link="link5"/>
-    <child link="grip_link_sub"/>
+    <child link="gripper_link_sub"/>
     <origin xyz="0.04225 -0.015 0" rpy="0 0 0"/>
     <axis xyz="0 0 1"/>
     <limit velocity="4.8" effort="1" lower="-0.7133010663668231" upper="1.059980724428978" />
-    <mimic joint="grip_joint" multiplier="-1"/>
+    <mimic joint="gripper" multiplier="-1"/>
   </joint>
   <!-- Transmission 6 -->
