Commit message: Minor fixes

File: open_manipulator_description/urdf/open_manipulator.gazebo.xacro (robot description, xacro)
@@ -37,5 +37,5 @@
   <gazebo>
     <plugin name="gazebo_ros_control" filename="libgazebo_ros_control.so">
-      <robotNamespace>open_manipulator</robotNamespace>
+      <robotNamespace>mikata_arm</robotNamespace>
       <controlPeriod>0.001</controlPeriod>
       <robotSimType>gazebo_ros_control/DefaultRobotHWSim</robotSimType>

File: open_manipulator_description/urdf/open_manipulator.urdf.xacro (robot description, xacro)
@@ -31,5 +31,5 @@
   <link name="link1">
     <visual>
-      <origin xyz="0 0 0" rpy="0 0 ${-pi*0.5}"/>
+      <origin xyz="0 0 0" rpy="0 0 0"/>
       <geometry>
         <mesh filename="package://open_manipulator_description/meshes/chain_link1.stl"/>
